File: Hardware/Power.sch (KiCad schematic (older format))
At the start: 17 parts, among them J5 Vin, U16 LM2675, U17 ADP3338AKCZ

Commit message: Add files via upload
HW layout and libs
Changed lines of the file:
@@
 LIBS:L298N
 LIBS:WS2812B
+LIBS:a4973
 LIBS:a3968
 LIBS:lm2675
@@
 $EndComp
 $Comp
-L GND #PWR082
+L GND #PWR086
 U 1 1 5A7063D6
 P 2200 2650
-F 0 "#PWR082" H 2200 2400 50  0001 C CNN
+F 0 "#PWR086" H 2200 2400 50  0001 C CNN
 F 1 "GND" H 2205 2477 50  0000 C CNN
 F 2 "" H 2200 2650 50  0001 C CNN
@@
 $EndComp
 $Comp
-L +24V #PWR083
+L +24V #PWR087
 U 1 1 5A7063DC
 P 2750 2350
-F 0 "#PWR083" H 2750 2200 50  0001 C CNN
+F 0 "#PWR087" H 2750 2200 50  0001 C CNN
 F 1 "+24V" H 2765 2523 50  0000 C CNN
 F 2 "" H 2750 2350 50  0001 C CNN
@@
 $EndComp
 $Comp
-L PWR_FLAG #FLG084
+L PWR_FLAG #FLG088
 U 1 1 5A7063E8
 P 8950 2800
-F 0 "#FLG084" H 8950 2875 50  0001 C CNN
+F 0 "#FLG088" H 8950 2875 50  0001 C CNN
 F 1 "PWR_FLAG" H 8950 2974 50  0000 C CNN
 F 2 "" H 8950 2800 50  0001 C CNN
@@
 $EndComp
 $Comp
-L GND #PWR085
+L GND #PWR089
 U 1 1 5A7063F5
 P 2750 2950
-F 0 "#PWR085" H 2750 2700 50  0001 C CNN
+F 0 "#PWR089" H 2750 2700 50  0001 C CNN
 F 1 "GND" H 2755 2777 50  0000 C CNN
 F 2 "" H 2750 2950 50  0001 C CNN
@@
 Connection ~ 5450 2750
 $Comp
-L GND #PWR086
+L GND #PWR090
 U 1 1 5A706428
 P 5450 3200
-F 0 "#PWR086" H 5450 2950 50  0001 C CNN
+F 0 "#PWR090" H 5450 2950 50  0001 C CNN
 F 1 "GND" H 5455 3027 50  0000 C CNN
 F 2 "" H 5450 3200 50  0001 C CNN
@@
 $EndComp
 $Comp
-L GND #PWR087
+L GND #PWR091
 U 1 1 5A706437
 P 6050 3200
-F 0 "#PWR087" H 6050 2950 50  0001 C CNN
+F 0 "#PWR091" H 6050 2950 50  0001 C CNN
 F 1 "GND" H 6055 3027 50  0000 C CNN
 F 2 "" H 6050 3200 50  0001 C CNN
@@
 Connection ~ 6050 2750
 $Comp
-L GND #PWR088
+L GND #PWR092
 U 1 1 5A706441
 P 4050 2900
-F 0 "#PWR088" H 4050 2650 50  0001 C CNN
+F 0 "#PWR092" H 4050 2650 50  0001 C CNN
 F 1 "GND" H 4055 2727 50  0000 C CNN
 F 2 "" H 4050 2900 50  0001 C CNN
@@
 $EndComp
 $Comp
-L GND #PWR089
+L GND #PWR093
 U 1 1 5A70646F
 P 6100 2200
-F 0 "#PWR089" H 6100 1950 50  0001 C CNN
+F 0 "#PWR093" H 6100 1950 50  0001 C CNN
 F 1 "GND" H 6105 2027 50  0000 C CNN
 F 2 "" H 6100 2200 50  0001 C CNN
@@
 $EndComp
 $Comp
-L GND #PWR090
+L GND #PWR094
 U 1 1 5A706496
 P 7550 3300
-F 0 "#PWR090" H 7550 3050 50  0001 C CNN
+F 0 "#PWR094" H 7550 3050 50  0001 C CNN
 F 1 "GND" H 7555 3127 50  0000 C CNN
 F 2 "" H 7550 3300 50  0001 C CNN
@@
 $EndComp
 $Comp
-L GND #PWR091
+L GND #PWR095
 U 1 1 5A70649C
 P 7100 3300
-F 0 "#PWR091" H 7100 3050 50  0001 C CNN
+F 0 "#PWR095" H 7100 3050 50  0001 C CNN
 F 1 "GND" H 7105 3127 50  0000 C CNN
 F 2 "" H 7100 3300 50  0001 C CNN
@@
 $EndComp
 $Comp
-L GND #PWR092
+L GND #PWR096
 U 1 1 5A7064A2
 P 8000 3250
-F 0 "#PWR092" H 8000 3000 50  0001 C CNN
+F 0 "#PWR096" H 8000 3000 50  0001 C CNN
 F 1 "GND" H 8005 3077 50  0000 C CNN
 F 2 "" H 8000 3250 50  0001 C CNN
@@
 	8250 2850 8250 2700
 $Comp
-L GND #PWR093
+L GND #PWR097
 U 1 1 5A7064C3
 P 8950 2850
-F 0 "#PWR093" H 8950 2600 50  0001 C CNN
+F 0 "#PWR097" H 8950 2600 50  0001 C CNN
 F 1 "GND" H 8955 2677 50  0000 C CNN
 F 2 "" H 8950 2850 50  0001 C CNN
@@
 	8000 2900 8000 2850
 Wire Wire Line
-	7100 2750 7100 2950
+	7100 2550 7100 2950
 Connection ~ 6350 2750
 $Comp
-L PWR_FLAG #FLG095
+L PWR_FLAG #FLG098
 U 1 1 5A7063E2
 P 9000 2050
-F 0 "#FLG095" H 9000 2125 50  0001 C CNN
+F 0 "#FLG098" H 9000 2125 50  0001 C CNN
 F 1 "PWR_FLAG" H 9000 2224 50  0000 C CNN
 F 2 "" H 9000 2050 50  0001 C CNN
@@
 	7950 2850 8250 2850
 $Comp
-L +5V #PWR?
-U 1 1 5A712DE9
-P 7100 2750
-F 0 "#PWR?" H 7100 2600 50  0001 C CNN
-F 1 "+5V" H 7100 2890 50  0000 C CNN
-F 2 "" H 7100 2750 50  0001 C CNN
-F 3 "" H 7100 2750 50  0001 C CNN
-	1    7100 2750
-	1    0    0    -1
-$EndComp
-$Comp
-L +3.3V #PWR?
+L +3.3V #PWR099
 U 1 1 5A712E1F
 P 8250 2700
-F 0 "#PWR?" H 8250 2550 50  0001 C CNN
+F 0 "#PWR099" H 8250 2550 50  0001 C CNN
 F 1 "+3.3V" H 8250 2840 50  0000 C CNN
 F 2 "" H 8250 2700 50  0001 C CNN
@@
 	1    0    0    -1
 $EndComp
+Connection ~ 7100 2750
+$Comp
+L VDD #PWR0100
+U 1 1 5A7C24FD
+P 7100 2550
+F 0 "#PWR0100" H 7100 2400 50  0001 C CNN
+F 1 "+5V" H 7100 2700 50  0000 C CNN
+F 2 "" H 7100 2550 50  0001 C CNN
+F 3 "" H 7100 2550 50  0001 C CNN
+	1    7100 2550
+	1    0    0    -1
+$EndComp

Commit message: Add files via upload
Parts:
- U16: symbol LM2675 -> LM2675-RESCUE-dispenser
Changed lines of the file:
@@
 LIBS:L298N
 LIBS:WS2812B
-LIBS:a4973
 LIBS:a3968
 LIBS:lm2675
@@
 	6350 3150 6350 3050
 $Comp
-L LM2675 U16
+L LM2675-RESCUE-dispenser U16
 U 1 1 5A7064D5
 P 3750 2700
