File: Hardware/dispenser.kicad_pcb (KiCad board)
At the start: 2 copper layers, 98 parts, among them J1 RJ45, J2 LCD4x20, J3 Motor2_con, J4 Motor1_con, J5 Vin, U1 PC817, U10 74HC14, U11 74HC14, U12 MCP4725, U13 ina219, U14 A3968, U15 74HC14, U16 LM2675, U17 ADP3338AKCZ, U2 PC817, U3 PC817, U4 PC817, U5 PC817, U6 PC817, U8 74HC14, U9 BluePill_STM32F103C

Commit message: Add files via upload
HW layout and libs
Parts:
- 1U10, 1U11, 1U12, 1U8, 1U9, C10, C9, D2, D3, D4, D5, R2, R24, R25, R26, R27, R3, R4, R5, U1, U12, U13, U14, U2, U3, U4, U5, U6: moved to F.Cu
- 1U13, C11, C12, C13, D14, L1, R28, R29, U16: moved to B.Cu
- moved J4 558.9 mm to (-103.4, -186.4), turned to 0 degrees
- moved J3 526.8 mm to (-103.4, -169.2), turned to 0 degrees
- moved 1U8 522.9 mm to (-67.5, -163.6), turned to 0 degrees
- moved U14 510.6 mm to (-80.1, -184.0), turned to 0 degrees
- moved U15 505.4 mm to (-82.0, -168.7), turned to 0 degrees
- moved 1U11 502.8 mm to (-67.5, -170.8), turned to 0 degrees
- moved 1U10 495.0 mm to (-74.0, -163.6), turned to 0 degrees
- moved 1U12 491.4 mm to (-74.0, -170.8), turned to 0 degrees
- moved C10 490.0 mm to (-67.0, -186.9), turned to 0 degrees
- moved U12 489.5 mm to (-56.1, -187.4), turned to 0 degrees
- moved R26 489.0 mm to (-60.8, -164.8)
- moved U13 488.6 mm to (-83.2, -157.2), turned to 0 degrees
- moved R24 488.6 mm to (-69.1, -178.1)
- moved R25 484.0 mm to (-76.3, -156.5), turned to 0 degrees
- moved R27 483.8 mm to (-69.5, -156.5)
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Connections:
- 1U1 pad 1: VCC -> +3V3
- 1U10 pad 1: +5V -> VDD
- 1U6 pad 1: VCC -> +3V3
- 1U7 pad 1: VCC -> +3V3
- C14 pad 1: +5V -> VDD
- C15 pad 1: +5V -> VDD
- C16 pad 1: +5V -> VDD
- D1 pad 3: VCC -> +3V3
- J1 pad 7: (no net) -> Net-(J1-Pad7)
- J2 pad 1: VCC -> +3V3
- L1 pad 2: +5V -> VDD
- R1 pad 1: VCC -> +3V3
- R19 pad 1: VCC -> +3V3
- R20 pad 1: VCC -> +3V3
- R21 pad 1: VCC -> +3V3
- R28 pad 1: +5V -> VDD
- U10 pad 14: +5V -> +3V3
- U11 pad 14: (no net) -> +3V3
- U11 pad 7: (no net) -> GND
- U14 pad 10: +5V -> VDD
- U17 pad 3: +5V -> VDD
- U5 pad 1: (no net) -> Net-(J1-Pad7)
- U9 pad 11: Net-(U10-Pad9) -> ENC_A_M1
- U9 pad 12: Net-(U10-Pad5) -> ENC_B_M1
- U9 pad 13: Net-(U10-Pad3) -> Limit_UPPER_M1
- U9 pad 14: Net-(U10-Pad1) -> Limit_LOWER_M1
- U9 pad 15: OUT_M1 -> Step_M1
- U9 pad 16: OUT_M2 -> CMD_M1
- U9 pad 22: Limit_LOWER_M1 -> Limit_LOWER_M2
- U9 pad 23: Limit_UPPER_M1 -> OUT_M2
- U9 pad 24: Limit_LOWER_M2 -> OUT_M1
- U9 pad 25: ENC_A_M2 -> Net-(U10-Pad5)
- U9 pad 26: ENC_B_M1 -> (no net)
- U9 pad 27: ENC_A_M1 -> Net-(U10-Pad9)
- U9 pad 28: ENC_B_M2 -> Step_M2
- U9 pad 29: (no net) -> CMD_M2
- U9 pad 30: CMD_M1 -> LED
- U9 pad 31: Step_M1 -> (no net)
- U9 pad 32: Step_M2 -> (no net)
- U9 pad 33: CMD_M2 -> (no net)
- U9 pad 36: (no net) -> Net-(U10-Pad1)
- U9 pad 37: (no net) -> Net-(U10-Pad3)
- U9 pad 5: Rot_Enc_B -> Rot_Enc_A
- U9 pad 6: Rot_Enc_A -> Rot_Enc_B
- U9 pad 7: (no net) -> Rot_Enc_SW
- U9 pad 8: (no net) -> ENC_A_M2
- U9 pad 9: Rot_Enc_SW -> ENC_B_M2
Routing:
- net +5V: track 45.3 -> 0.00 mm
- net VDD: track 0.00 -> 42.0 mm, vias 0 -> 1
- net /MotorDriver/M2B: track 41.5 -> 0.00 mm
- net Net-(J3-Pad7): track 33.9 -> 0.00 mm, vias 1 -> 0
- net /MotorDriver/M1B: track 31.6 -> 0.00 mm
- net /MotorDriver/M2A: track 30.6 -> 0.00 mm
- net Net-(C10-Pad1): track 26.0 -> 0.00 mm
- net Net-(J1-Pad3): track 24.4 -> 0.00 mm
- net GND: track 23.1 -> 0.00 mm
- net Net-(J1-Pad4): track 20.0 -> 0.00 mm
- net Net-(J1-Pad8): track 19.8 -> 0.00 mm
- net /MotorDriver/M1A: track 18.9 -> 0.00 mm
- net +24V: track 46.9 -> 28.9 mm, vias 1 -> 0
- net +3V3: track 19.1 -> 5.77 mm
- net SDA: track 12.4 -> 0.00 mm
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- removed copper zone on B.Cu, net GNDD

Commit message: Add files via upload
Parts:
- 1U2, C2, C3, C4, C5, D6, D7, D8, D9, R10, R11, R12, R13, R14, R15, R8, R9, U8: moved to B.Cu
- moved R4 116.3 mm to (103.6, 67.1), turned to 270 degrees
- moved R3 103.9 mm to (103.6, 94.5), turned to 270 degrees
- moved R6 95.8 mm to (127.0, 84.8)
- moved R7 87.8 mm to (127.0, 79.2)
- moved R5 83.0 mm to (103.6, 89.4), turned to 270 degrees
- moved R15 78.8 mm to (140.7, 63.0)
- moved R12 78.4 mm to (141.2, 98.6)
- moved R9 78.3 mm to (140.7, 68.6)
- moved C3 75.4 mm to (140.7, 75.2), turned to 180 degrees
- moved D6 72.6 mm to (141.2, 96.0), turned to 180 degrees
- moved R10 71.4 mm to (141.2, 80.8)
- moved D8 69.8 mm to (141.2, 83.3), turned to 180 degrees
- moved R13 64.7 mm to (140.7, 73.2)
- moved R14 59.2 mm to (141.2, 85.9)
- moved R8 55.9 mm to (141.2, 93.5)
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Routing:
- net Net-(J1-Pad3): track 0.00 -> 29.9 mm, vias 0 -> 1
- net +24Logic: track 0.00 -> 27.8 mm, vias 0 -> 1
- net Net-(J1-Pad7): track 0.00 -> 20.8 mm, vias 0 -> 1
- net Net-(J1-Pad4): track 0.00 -> 20.6 mm, vias 0 -> 1
- net Net-(J1-Pad8): track 0.00 -> 20.0 mm, vias 0 -> 1
- net Net-(J1-Pad6): track 0.00 -> 17.0 mm, vias 0 -> 1
- net Net-(J1-Pad2): track 10.0 -> 16.7 mm, vias 0 -> 1
- net GNDD: track 0.00 -> 6.49 mm, vias 0 -> 1
- net Net-(D6-Pad2): track 0.00 -> 6.24 mm
- net Net-(D8-Pad2): track 0.00 -> 6.24 mm
- net Net-(D4-Pad2): track 0.00 -> 6.16 mm
- net Net-(D5-Pad2): track 0.00 -> 6.11 mm
- net Net-(D9-Pad2): track 0.00 -> 6.10 mm
- net Net-(D2-Pad2): track 0.00 -> 6.10 mm
- net Net-(D3-Pad2): track 0.21 -> 6.10 mm
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- added copper zone on B.Cu, net GNDD
- added copper zone on F.Cu, net GNDD
Other:
- net class alla andra: clearance 0.2 -> 0.3

Commit message: Layout - some pin changes to 74hc14
Parts:
- 1U10, 1U11, 1U12, 1U8, 1U9, C9, R24, R25, R26, R27, U10, U12, U13, U14: moved to B.Cu
- moved J3 428.1 mm to (224.2, 106.4), turned to 90 degrees
- moved 1U12 415.2 mm to (230.1, 111.9), turned to 270 degrees
- moved J4 413.5 mm to (224.2, 66.0), turned to 90 degrees
- moved U14 396.6 mm to (209.7, 86.8)
- moved U15 387.7 mm to (210.6, 85.7)
- moved C9 384.4 mm to (222.3, 84.8), turned to 270 degrees
- moved 1U11 383.1 mm to (229.4, 71.3), turned to 270 degrees
- moved R25 382.2 mm to (220.2, 84.8), turned to 270 degrees
- moved 1U10 378.5 mm to (216.5, 78.9)
- moved C10 375.6 mm to (201.5, 75.8), turned to 90 degrees
- moved R24 372.6 mm to (196.2, 83.5)
- moved U12 371.1 mm to (202.9, 78.4), turned to 180 degrees
- moved R27 366.4 mm to (211.8, 78.2), turned to 90 degrees
- moved U13 365.7 mm to (196.2, 78.7)
- moved R26 362.6 mm to (200.7, 86.3), turned to 180 degrees
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Connections:
- U10 pad 10: (no net) -> Motor_Input_2B
- U10 pad 11: (no net) -> Net-(U10-Pad11)
- U10 pad 2: Motor_Input_1A -> Motor_Input_1B
- U10 pad 4: Motor_Input_1B -> Motor_Input_1A
- U10 pad 5: Net-(U10-Pad5) -> (no net)
- U10 pad 6: Motor_Input_2A -> (no net)
- U10 pad 8: Motor_Input_2B -> Motor_Input_2A
- U9 pad 25: Net-(U10-Pad5) -> Net-(U10-Pad11)
- U9 pad 36: Net-(U10-Pad1) -> Net-(U10-Pad3)
- U9 pad 37: Net-(U10-Pad3) -> Net-(U10-Pad1)
Routing:
- net Limit_UPPER_M1: track 0.00 -> 148.7 mm, vias 0 -> 2
- net Limit_LOWER_M1: track 0.00 -> 148.6 mm, vias 0 -> 2
- net ENC_B_M2: track 0.00 -> 110.5 mm, vias 0 -> 1
- net ENC_B_M1: track 0.00 -> 104.6 mm, vias 0 -> 1
- net GND: track 0.00 -> 91.0 mm, vias 0 -> 1
- net ENC_A_M2: track 0.00 -> 61.5 mm, vias 0 -> 1
- net +3V3: track 5.77 -> 65.3 mm, vias 0 -> 1
- net Limit_LOWER_M2: track 0.00 -> 50.5 mm
- net OUT_M1: track 0.00 -> 48.9 mm, vias 0 -> 1
- net OUT_M2: track 0.00 -> 48.9 mm, vias 0 -> 1
- net Limit_upper_M2: track 0.00 -> 47.3 mm
- net Step_M2: track 0.00 -> 43.4 mm, vias 0 -> 2
- net VDD: track 42.0 -> 84.0 mm, vias 1 -> 2
- net Net-(J3-Pad7): track 0.00 -> 41.6 mm, vias 0 -> 1
- net /MotorDriver/M1B: track 0.00 -> 39.6 mm
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Other:
- net class 24v: clearance 0.5 -> 0.3
- net class 5v: clearance 0.2 -> 0.3
- net class Default: clearance 0.15 -> 0.25
- rule trace_clearance: 0.15 -> 0.25

Commit message: Add files via upload
Parts:
- moved 1U13 231.8 mm to (339.7, 32.3)
- moved C11 231.8 mm to (335.9, 30.2)
- moved C12 231.8 mm to (331.3, 30.2)
- moved C15 231.8 mm to (337.9, 30.5)
- moved C16 231.8 mm to (348.6, 15.7)
- moved D13 231.8 mm to (320.0, 19.9)
- moved C13 231.8 mm to (346.7, 24.8)
- moved C17 231.8 mm to (337.8, 16.3)
- moved D14 231.8 mm to (334.0, 20.4)
- moved F1 231.8 mm to (324.9, 27.2)
- moved J5 231.8 mm to (317.6, 27.1)
- moved L1 231.8 mm to (347.6, 19.7)
- moved R28 231.8 mm to (353.7, 27.5)
- moved R29 231.8 mm to (356.1, 27.5)
- moved U16 231.8 mm to (346.2, 29.3)
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Routing:
- net ENC_A_M1: track 21.5 -> 82.2 mm, vias 0 -> 1
- net Limit_UPPER_M1: track 148.7 -> 103.7 mm, vias 2 -> 0
- net Limit_LOWER_M1: track 148.6 -> 112.8 mm, vias 2 -> 0
- net VDD: track 84.0 -> 50.1 mm, vias 2 -> 1
- net +3V3: track 65.3 -> 94.2 mm
- net Rot_Enc_SW: track 0.00 -> 26.5 mm
- net Rot_Enc_B: track 0.00 -> 23.3 mm
- net ENC_B_M1: track 104.6 -> 82.6 mm
- net OUT_M2: track 48.9 -> 27.4 mm
- net Rot_Enc_A: track 0.00 -> 20.2 mm
- net OUT_M1: track 48.9 -> 29.6 mm
- net SCL: track 31.4 -> 13.9 mm, vias 0 -> 1
- net SDA: track 28.3 -> 11.1 mm, vias 0 -> 1
- net CMD_M2: track 38.7 -> 55.0 mm, vias 0 -> 2
- net CMD_M1: track 27.4 -> 43.3 mm, vias 0 -> 2
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Other:
- net class Default: clearance 0.25 -> 0.3
- rule trace_clearance: 0.25 -> 0.3

Commit message: Add files via upload
Parts:
- removed C14: 68Uf, Capacitors_SMD:CP_Elec_10x10
- 1U8, C11, C12, D13: moved to F.Cu
- moved 1U1 333.2 mm to (201.2, 93.7), turned to 270 degrees
- moved D1 329.6 mm to (196.7, 94.8), turned to 270 degrees
- moved JP1 320.7 mm to (164.7, 128.8), turned to 90 degrees
- moved C1 310.8 mm to (167.0, 135.5)
- moved R1 303.9 mm to (167.0, 133.1)
- moved U17 176.1 mm to (170.8, 52.3)
- moved C16 175.3 mm to (177.9, 55.3), turned to 0 degrees
- moved C17 174.9 mm to (168.8, 61.1)
- moved L1 167.2 mm to (183.6, 52.6), turned to 180 degrees
- moved R28 165.6 mm to (190.8, 57.4), turned to 0 degrees
- moved R29 161.5 mm to (197.4, 57.4), turned to 180 degrees
- moved C13 158.9 mm to (190.8, 55.4)
- moved U16 151.4 mm to (196.5, 51.9), turned to 0 degrees
- moved C15 147.2 mm to (191.6, 47.1), turned to 0 degrees
- moved D14 144.6 mm to (191.5, 44.7)
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Connections:
- 1U1 pad 1: +3V3 -> VDD
- D1 pad 3: +3V3 -> VDD
- J2 pad 1: +3V3 -> VDD
Routing:
- net +3V3: track 94.2 -> 134.6 mm, vias 1 -> 2
- net LED: track 0.00 -> 25.4 mm, vias 0 -> 1
- net GND: track 104.4 -> 95.0 mm, vias 4 -> 3
- net SCL: track 13.9 -> 22.6 mm, vias 1 -> 2
- net Net-(C10-Pad1): track 20.7 -> 29.0 mm
- net SDA: track 11.1 -> 18.0 mm, vias 1 -> 2
- net Net-(R28-Pad2): track 7.85 -> 14.6 mm
- net ENC_B_M2: track 117.8 -> 113.3 mm
- net Net-(U10-Pad3): track 21.3 -> 19.6 mm
- net +24V: track 32.9 -> 31.5 mm, vias 0 -> 1
- net Net-(C13-Pad2): track 3.34 -> 1.92 mm
- net VDD: track 50.1 -> 48.8 mm
- net Net-(J3-Pad7): track 41.6 -> 40.7 mm
- net Net-(J4-Pad2): track 24.9 -> 24.2 mm
- net /MotorDriver/M1B: track 39.7 -> 40.4 mm
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Other:
- net class 24v: clearance 0.3 -> 0.2
- net class Default: clearance 0.3 -> 0.2
- rule trace_clearance: 0.3 -> 0.2

Commit message: Add files via upload
Parts:
- removed 1U6, 1U7: 0,1U, Capacitors_SMD:C_0805_HandSoldering
- removed C6, C7, C8: 0.1uF, Capacitors_SMD:C_0805_HandSoldering
- removed D10, D11, D12: 1m4148, Diodes_SMD:D_MiniMELF_Handsoldering
- removed R18, R19, R20, R21, R22, R23: 10K, Resistors_SMD:R_0805_HandSoldering
- removed ROT1: ROTARY-ENCODER, Libs:ROTARY-ENCODER-Ebay
- removed U11: 74HC14, Housings_SOIC:SOIC-14_3.9x8.7mm_Pitch1.27mm
- 1U5, C16: moved to B.Cu
- J2: value LCD4x20 -> LCD_and_RotEnc; footprint Pin_Headers:Pin_Header_Straight_1x04_Pitch2.54mm -> Pin_Headers:Pin_Header_Straight_1x07_Pitch2.54mm
- moved 1U4 164.1 mm to (158.4, 116.9), turned to 270 degrees
- moved 1U3 150.3 mm to (160.7, 116.8), turned to 270 degrees
- moved 1U5 116.8 mm to (179.9, 71.9), turned to 270 degrees
- moved R17 104.5 mm to (192.7, 84.4), turned to 180 degrees
- moved R16 87.0 mm to (192.7, 86.8), turned to 180 degrees
- moved J2 10.0 mm to (162.5, 42.9), turned to 0 degrees
- moved R27 7.12 mm to (220.4, 68.6), turned to 0 degrees
- moved C16 5.33 mm to (173.6, 52.1), turned to 180 degrees
- moved C17 2.12 mm to (167.3, 59.6), turned to 180 degrees
- moved 1U10 2.11 mm to (220.1, 70.6)
Connections:
- 1U1 pad 1: VDD -> +3V3
- D1 pad 3: VDD -> +3V3
- J2 pad 2: SCL -> SDA
- J2 pad 3: SDA -> SCL
- J2 pad 4: GND -> Rot_Enc_SW
Routing:
- net +3V3: track 134.6 -> 347.1 mm, vias 2 -> 7
- net VDD: track 48.8 -> 194.6 mm, vias 1 -> 3
- net SCL: track 22.6 -> 115.4 mm, vias 2 -> 3
- net SDA: track 18.0 -> 110.2 mm, vias 2 -> 3
- net Rot_Enc_SW: track 26.5 -> 38.9 mm
- net +24V: track 31.5 -> 42.5 mm, vias 1 -> 3
- net Rot_Enc_A: track 20.2 -> 30.6 mm
- net Rot_Enc_B: track 23.3 -> 32.1 mm
- net Net-(R27-Pad1): track 8.97 -> 15.1 mm
- net GND: track 95.0 -> 100.5 mm
- net ENC_B_M2: track 113.3 -> 109.1 mm
- net +24Logic: track 28.1 -> 31.3 mm
- net Net-(C10-Pad1): track 29.0 -> 31.6 mm
- net Net-(J1-Pad6): track 17.0 -> 19.0 mm
- net Net-(C4-Pad1): track 23.7 -> 25.3 mm
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Other:
- net class Default: clearance 0.2 -> 0.4
- rule trace_clearance: 0.2 -> 0.4

Commit message: Add files via upload
Parts:
- removed C15: 120Uf, Capacitors_SMD:CP_Elec_10x10
- added C14: 68Uf, Capacitors_SMD:CP_Elec_10x10, F.Cu at (174.1, 146.2)
- 1U13, 1U2, 1U5, C13, C16, C2, C3, C4, C5, D14, D6, D7, D8, D9, L1, R10, R11, R12, R13, R14, R15, R28, R29, R8, R9, U10, U16, U8: moved to F.Cu
- 1U8, C10: moved to B.Cu
- moved R8 356.0 mm to (553.9, 159.7), turned to 0 degrees
- moved R6 348.5 mm to (540.4, 159.7), turned to 0 degrees
- moved R9 348.0 mm to (549.3, 145.5), turned to 0 degrees
- moved R11 347.5 mm to (549.3, 138.4), turned to 0 degrees
- moved R10 340.6 mm to (540.4, 152.6), turned to 0 degrees
- moved R14 337.1 mm to (542.5, 145.5), turned to 0 degrees
- moved R7 337.1 mm to (529.0, 164.1), turned to 0 degrees
- moved R4 336.7 mm to (553.9, 152.6), turned to 0 degrees
- moved D2 335.3 mm to (549.1, 131.3), turned to 0 degrees
- moved C3 334.3 mm to (542.4, 131.3), turned to 0 degrees
- moved 1U2 332.8 mm to (520.2, 157.1), turned to 0 degrees
- moved R5 331.7 mm to (547.1, 152.6), turned to 0 degrees
- moved R2 330.7 mm to (547.1, 159.7), turned to 0 degrees
- moved D8 329.8 mm to (533.5, 131.3), turned to 0 degrees
- moved D7 329.5 mm to (533.5, 138.5), turned to 0 degrees
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Connections:
- J2 pad 1: VDD -> +3V3
- J3 pad 5: /MotorDriver/M2A -> /MotorDriver/M2B
- J3 pad 9: /MotorDriver/M2B -> /MotorDriver/M2A
Routing:
- net +3V3: track 347.1 -> 61.5 mm, vias 7 -> 0
- net VDD: track 194.6 -> 39.3 mm, vias 3 -> 0
- net SCL: track 115.4 -> 0.00 mm, vias 3 -> 0
- net SDA: track 110.2 -> 0.00 mm, vias 3 -> 0
- net Limit_LOWER_M1: track 113.0 -> 12.2 mm
- net GND: track 100.5 -> 0.00 mm, vias 3 -> 0
- net ENC_B_M2: track 109.1 -> 11.9 mm, vias 1 -> 0
- net Limit_UPPER_M1: track 104.1 -> 10.1 mm
- net ENC_A_M1: track 81.7 -> 6.14 mm, vias 1 -> 0
- net ENC_B_M1: track 81.0 -> 9.26 mm, vias 1 -> 0
- net ENC_A_M2: track 74.3 -> 12.1 mm, vias 1 -> 0
- net CMD_M2: track 55.0 -> 0.00 mm, vias 2 -> 0
- net Step_M2: track 54.1 -> 0.00 mm
- net Step_M1: track 44.0 -> 0.00 mm, vias 2 -> 0
- net CMD_M1: track 42.1 -> 0.00 mm, vias 2 -> 0
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- removed copper zone on B.Cu, net GND
- removed copper zone on F.Cu, net GND
- removed copper zone on B.Cu, net GNDD
- removed copper zone on F.Cu, net GNDD
Other:
- net class 24v: clearance 0.2 -> 0.3
- net class Default: clearance 0.4 -> 0.3
- net class GNDD: clearance 1 -> 0.3
- rule trace_clearance: 0.4 -> 0.3

Commit message: one motor
Parts:
- removed C1: 0,1u, Capacitors_SMD:C_0805_HandSoldering
- removed C3, C5: 0.1uF, Capacitors_SMD:C_0805_HandSoldering
- removed D3, D5: LED, LEDs:LED_0805_HandSoldering
- removed D7: 1m4148, Diodes_SMD:D_MiniMELF_Handsoldering
- removed D9: 1n4148, Diodes_SMD:D_MiniMELF_Handsoldering
- removed J3: Motor2_con, Libs:Dsub9
- removed JP1: Jumper, Pin_Headers:Pin_Header_Straight_1x03_Pitch2.54mm
- removed R1, R11, R13, R15, R9: 10K, Resistors_SMD:R_0805_HandSoldering
- removed R2, R4: 1K, Resistors_SMD:R_0805_HandSoldering
- removed R7: 120R, Resistors_SMD:R_0805_HandSoldering
- removed U10: 74HC14, Housings_SOIC:SOIC-14_3.9x8.7mm_Pitch1.27mm
- removed U2, U4, U6: PC817, Libs:817opto
- added C15: 120Uf, Capacitors_SMD:CP_Elec_10x10, F.Cu at (127.4, 46.0)
- added REF**: JUMPER 5MM, Libs:JUMPER_5MM, F.Cu at (132.4, 96.2)
- 1U1, 1U2, 1U5, C2, C4, D2, D4, D6, D8, R10, R12, R14, R3, R5, R6, R8, U1, U15, U3, U5, U8: moved to B.Cu
- 1U11: moved to F.Cu
- moved R5 429.9 mm to (128.2, 56.4), turned to 180 degrees
- moved D2 423.0 mm to (133.2, 54.1)
- moved R3 417.3 mm to (128.2, 54.1), turned to 180 degrees
- moved R8 413.6 mm to (150.0, 70.5), turned to 180 degrees
- moved R6 404.8 mm to (143.9, 78.1), turned to 270 degrees
- moved D4 404.5 mm to (133.3, 56.4)
- moved R14 401.5 mm to (150.5, 59.0)
- moved J1 401.2 mm to (129.1, 62.1), turned to 270 degrees
- moved R10 400.4 mm to (150.5, 61.5)
- moved D8 390.1 mm to (150.8, 55.6), turned to 180 degrees
- moved R12 382.2 mm to (152.5, 67.5)
- moved 1U2 379.9 mm to (149.5, 74.4), turned to 270 degrees
- moved C4 379.6 mm to (153.6, 51.7), turned to 90 degrees
- moved D6 370.2 mm to (152.8, 64.9), turned to 180 degrees
- moved C2 366.8 mm to (156.6, 62.4)
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Connections:
- 1U1 pad 1: +3V3 -> VDD
- 1U11 pad 1: +3V3 -> VDD
- D1 pad 3: +3V3 -> VDD
- J1 pad 2: Net-(J1-Pad2) -> (no net)
- J1 pad 3: Net-(J1-Pad3) -> (no net)
- J1 pad 4: Net-(J1-Pad4) -> (no net)
- J2 pad 1: +3V3 -> VDD
- J4 pad 3: (no net) -> Net-(J4-Pad3)
- J4 pad 4: Limit_UPPER_M1 -> (no net)
- J4 pad 8: Limit_LOWER_M1 -> Net-(J4-Pad8)
- U14 pad 11: /MotorDriver/M2B -> (no net)
- U14 pad 14: Motor_Input_2B -> (no net)
- U14 pad 15: Motor_Input_2A -> (no net)
- U14 pad 16: /MotorDriver/M2A -> (no net)
- U15 pad 1: Net-(J4-Pad7) -> Net-(J4-Pad2)
- U15 pad 2: ENC_A_M1 -> ENC_B_M1
- U15 pad 3: Net-(J4-Pad2) -> Net-(J4-Pad7)
- U15 pad 4: ENC_B_M1 -> ENC_A_M1
- U15 pad 5: Net-(J3-Pad7) -> Net-(J4-Pad3)
- U15 pad 6: ENC_A_M2 -> Limit_LOWER_M1
- U15 pad 8: ENC_B_M2 -> Limit_UPPER_M1
- U15 pad 9: Net-(J3-Pad2) -> Net-(J4-Pad8)
- U8 pad 5: Net-(C3-Pad1) -> (no net)
- U8 pad 6: CMD_M2 -> (no net)
- U8 pad 8: Step_M2 -> (no net)
- U8 pad 9: Net-(C5-Pad1) -> (no net)
- U9 pad 10: LED -> (no net)
- U9 pad 13: Limit_UPPER_M1 -> (no net)
- U9 pad 14: Limit_LOWER_M1 -> (no net)
- U9 pad 15: Step_M1 -> CMD_M1
- U9 pad 16: CMD_M1 -> Step_M1
- U9 pad 17: reset_in -> (no net)
- U9 pad 21: Limit_upper_M2 -> (no net)
- U9 pad 22: Limit_LOWER_M2 -> (no net)
- U9 pad 23: OUT_M2 -> (no net)
- U9 pad 25: Net-(U10-Pad11) -> Limit_UPPER_M1
- U9 pad 26: (no net) -> Limit_LOWER_M1
- U9 pad 27: Net-(U10-Pad9) -> (no net)
- U9 pad 28: Step_M2 -> (no net)
- U9 pad 29: CMD_M2 -> (no net)
- U9 pad 36: Net-(U10-Pad3) -> Motor_Input_1A
- U9 pad 37: Net-(U10-Pad1) -> Motor_Input_1B
- U9 pad 5: Rot_Enc_A -> Rot_Enc_B
- U9 pad 6: Rot_Enc_B -> Rot_Enc_A
- U9 pad 8: ENC_A_M2 -> (no net)
- U9 pad 9: ENC_B_M2 -> (no net)
Routing:
- net GND: track 0.00 -> 369.2 mm
- net +3V3: track 61.5 -> 258.4 mm, vias 0 -> 5
- net VDD: track 39.3 -> 225.0 mm, vias 0 -> 2
- net +24V: track 16.5 -> 199.3 mm, vias 0 -> 2
- net SCL: track 0.00 -> 100.7 mm, vias 0 -> 2
- net SDA: track 0.00 -> 96.9 mm, vias 0 -> 2
- net OUT_M1: track 0.00 -> 66.9 mm, vias 0 -> 2
- net ENC_A_M1: track 6.14 -> 61.4 mm
- net ENC_B_M1: track 9.26 -> 57.8 mm
- net Net-(J4-Pad8): track 0.00 -> 41.8 mm
- net Net-(J3-Pad7): track 38.9 -> 0.00 mm, vias 1 -> 0
- net Rot_Enc_SW: track 0.00 -> 37.1 mm
- net Net-(J4-Pad3): track 0.00 -> 33.4 mm
- net Rot_Enc_A: track 0.00 -> 33.3 mm
- net /MotorDriver/M2B: track 30.5 -> 0.00 mm
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- added copper zone on B.Cu, net GND
- added copper zone on F.Cu, net GND
- added copper zone on B.Cu, net GNDD
Other:
- board outline added: 100.1 x 68.8 mm
