File: Hardware/dispenser.kicad_pcb (KiCad board)
At the start: 2 copper layers, 100.1 x 68.8 mm, 62 parts, among them J1 RJ45, J2 LCD_and_RotEnc, J4 Motor1_con, J5 Vin, U1 PC817, U12 MCP4725, U13 ina219, U14 A3968, U15 74HC14, U16 LM2675, U17 ADP3338AKCZ, U3 PC817, U5 PC817, U8 74HC14, U9 BluePill_STM32F103C

Commit message: Getting there
Routing:
- net Net-(C9-Pad1): track 3.02 -> 5.37 mm
Changed lines of the file:
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@@
-(kicad_pcb (version 4) (host pcbnew 4.0.7)
+(kicad_pcb (version 4) (host pcbnew 4.0.5+dfsg1-4)
   (general
     (links 152)
@@
     (thickness 1.6)
     (drawings 6)
-    (tracks 584)
+    (tracks 586)
     (zones 0)
     (modules 62)
@@
   (segment (start 153.5244 55.626) (end 153.5244 57.4248) (width 0.4) (layer B.Cu) (net 28) (status 10))
   (segment (start 153.5244 57.4248) (end 151.9704 58.9788) (width 0.4) (layer B.Cu) (net 28) (status 20))
+  (segment (start 201.168 86.0768) (end 198.8604 86.0768) (width 0.4) (layer B.Cu) (net 29))
+  (segment (start 198.8604 86.0768) (end 198.8312 86.106) (width 0.4) (layer B.Cu) (net 29))
   (segment (start 198.9328 86.0044) (end 198.8312 86.106) (width 0.4) (layer B.Cu) (net 29) (status 30))
   (segment (start 198.8312 86.106) (end 198.8312 84.4822) (width 0.4) (layer B.Cu) (net 29) (status 10))
